Commit message: Created core URDF

File: description/inertial_macros.xacro (robot description, xacro)
@@ -8,6 +8,6 @@
             <mass value="${mass}" />
             <inertia ixx="${(2/5) * mass * (radius*radius)}" ixy="0.0" ixz="0.0"
-                    iyy="${(2/5) * mass * (radius*radius)}" iyz="0.0"
-                    izz="${(2/5) * mass * (radius*radius)}"/>
+                     iyy="${(2/5) * mass * (radius*radius)}" iyz="0.0"
+                     izz="${(2/5) * mass * (radius*radius)}"/>
         </inertial>
     </xacro:macro>
@@ -17,6 +17,6 @@
             <mass value="${mass}" />
             <inertia ixx="${(1/12) * mass * (y*y+z*z)}" ixy="0.0" ixz="0.0"
-                    iyy="${(1/12) * mass * (x*x+z*z)}" iyz="0.0"
-                    izz="${(1/12) * mass * (x*x+y*y)}"/>
+                     iyy="${(1/12) * mass * (x*x+z*z)}" iyz="0.0"
+                     izz="${(1/12) * mass * (x*x+y*y)}"/>
         </inertial>
     </xacro:macro>
@@ -26,6 +26,6 @@
             <mass value="${mass}" />
             <inertia ixx="${(1/12) * mass * (3*radius*radius + length*length)}" ixy="0.0" ixz="0.0"
-                    iyy="${(1/12) * mass * (3*radius*radius + length*length)}" iyz="0.0"
-                    izz="${(1/2) * mass * (radius*radius)}"/>
+                     iyy="${(1/12) * mass * (3*radius*radius + length*length)}" iyz="0.0"
+                     izz="${(1/2) * mass * (radius*radius)}"/>
         </inertial>
     </xacro:macro>

File: description/robot_core.xacro (robot description, xacro)
@@ -19,5 +19,5 @@
     <!--CHASSIS LINK-->
     <joint name="chassis_joint" type="fixed">
-        <parent link="base_link"/>
+        <p arent link="base_link"/>
         <child link="chassis"/>
         <origin xyz="-0.1 0 0"/>
